File: plates/3x6/pcb/plate.kicad_pcb (KiCad board)
At the start: 2 copper layers, 273.7 x 94.8 mm, 0 parts

Commit message: update plate
Other:
- board size 273.7 x 94.8 mm -> 272.9 x 94.4 mm

Commit message: update plate
Other:
- board size 272.9 x 94.4 mm -> 388.9 x 93.5 mm
