File: plates/3x6/pcb/plate.kicad_pcb (KiCad board)
At the start: 2 copper layers, 388.9 x 93.5 mm, 0 parts

Commit message: update plate
Other:
- board size 388.9 x 93.5 mm -> 390.2 x 93.6 mm

Commit message: update plate
Other:
- board size 390.2 x 93.6 mm -> 390.1 x 93.5 mm

Commit message: Update plate.kicad_pcb
Other:
- board size 390.1 x 93.5 mm -> 389.3 x 93.5 mm

Commit message: update plate
Other:
- board size 389.3 x 93.5 mm -> 408.2 x 93.5 mm

Commit message: update plate
Other:
- board size 408.2 x 93.5 mm -> 408 x 93.5 mm
